Commit message: fixed mesh paths

File: src/so_101_arm/urdf/so_101_arm_6dof.urdf (robot description, URDF)
Before this commit: robot so_101_arm, 8 links, 7 joints
Links:
- link base: geometry collision mesh filename=package://so_101_arm/models/so_101_arm/meshes/base_motor_ho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; collision mesh filename=package://so_101_arm/models/so_101_arm/meshes/base_so101_v2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
- link gripper: geometry collision mesh filename=package://so_101_arm/models/so_101_arm/meshes/sts3215_03a_v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; collision mesh filename=package://so_101_arm/models/so_101_arm/meshes/wrist_roll_fo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
- link lower_arm: geometry collision mesh filename=package://so_101_arm/models/so_101_arm/meshes/motor_holder_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; collision mesh filename=package://so_101_arm/models/so_101_arm/meshes/sts3215_03a_v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
- link moving_jaw: geometry collision mesh filename=package://so_101_arm/models/so_101_arm/meshes/moving_jaw_so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; visual mesh filename=package://so_101_arm/models/so_101_arm/meshes/moving_jaw_so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
- link shoulder: geometry collision mesh filename=package://so_101_arm/models/so_101_arm/meshes/motor_holder_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; collision mesh filename=package://so_101_arm/models/so_101_arm/meshes/rotation_pitc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
- link upper_arm: geometry collision mesh filename=package://so_101_arm/models/so_101_arm/meshes/sts3215_03a_v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; collision mesh filename=package://so_101_arm/models/so_101_arm/meshes/upper_arm_so1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
- link wrist: geometry collision mesh filename=package://so_101_arm/models/so_101_arm/meshes/sts3215_03a_n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; collision mesh filename=package://so_101_arm/models/so_101_arm/meshes/wrist_roll_pi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

Commit message: fix rviz gazebo conflict

File: src/so_101_arm/urdf/so_101_arm_6dof.urdf (robot description, URDF)
Before this commit: robot so_101_arm, 8 links, 7 joints
Links:
- link base: geometry collision box size=0.05 0.05 0.05; collision box size=0.06 0.06 0.02
- link gripper: geometry collision box size=0.04 0.04 0.03; collision cylinder length=0.04 radius=0.025
- link lower_arm: geometry collision box size=0.10 0.04 0.04; collision cylinder length=0.04 radius=0.025
- link moving_jaw: geometry collision box size=0.02 0.01 0.04; visual mesh filename=package://so_101_arm/models/so_101_arm/meshes/moving_jaw_so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
- link shoulder: geometry collision box size=0.04 0.04 0.06; collision cylinder length=0.04 radius=0.025
- link upper_arm: geometry collision box size=0.12 0.04 0.04; collision cylinder length=0.04 radius=0.025
- link wrist: geometry collision box size=0.05 0.05 0.06; collision cylinder length=0.04 radius=0.025
