Commit message: use xacro

File: src/so_101_arm/urdf/so_101_arm_6dof.urdf.xacro (robot description, xacro)
@@ -1,4 +1,8 @@
-<!-- SO-101 Robot Arm URDF -->
-<robot name="so_101_arm">
+<?xml version="1.0"?>
+<!-- SO-101 Robot Arm URDF.XACRO -->
+<robot xmlns:xacro="http://www.ros.org/wiki/xacro" name="so_101_arm">
+  <!-- XACRO Parameters -->
+  <xacro:arg name="controller_config_file" default="$(find so_101_arm)/config/controllers_6dof.yaml"/>
+  <xacro:property name="controller_config" value="$(arg controller_config_file)"/>
   <!-- ROS2 Control configuration -->
   <ros2_control name="gz_ros2_control/GazeboSimSystem" type="system">
@@ -63,5 +67,6 @@
   <gazebo>
     <plugin filename="gz_ros2_control-system" name="gz_ros2_control::GazeboSimROS2ControlPlugin">
-        <parameters>/home/rohan/projects/so-arm101_ws/install/so_101_arm/share/so_101_arm/config/controllers_6dof.yaml</parameters>
+        <!-- XACRO: Use parameterized controller config file -->
+        <parameters>${controller_config}</parameters>
         <robot_param>robot_description</robot_param>
         <robot_param_node>robot_state_publisher</robot_param_node>

Commit message: updated designs

File: src/so_101_arm/urdf/so_101_arm_6dof.urdf.xacro (robot description, xacro)
@@ -86,11 +86,11 @@
     <origin xyz="0 0 0" rpy="0 0 0"/>
   </joint>
-  <!-- Base link -->
+  <!-- Base link with INCREASED MASS to prevent falling -->
   <link name="base">
     <inertial>
       <origin xyz="0.020739 0.00204287 0.065966" rpy="0 0 0"/>
-      <mass value="0.147"/>
-      <inertia ixx="0.000136117" ixy="4.59787e-07" ixz="9.75275e-08"
-               iyy="0.000114686" iyz="-4.97151e-06" izz="0.000130364"/>
+      <mass value="50.0"/>  <!-- INCREASED from 0.147 to prevent falling -->
+      <inertia ixx="0.136117" ixy="4.59787e-06" ixz="9.75275e-07"
+               iyy="0.114686" iyz="-4.97151e-05" izz="0.130364"/>
     </inertial>
     <!-- Base motor holder visual -->

Commit message: try to attach arm to table mount

File: src/so_101_arm/urdf/so_101_arm_6dof.urdf.xacro (robot description, xacro)
@@ -86,5 +86,5 @@
     <origin xyz="0 0 0" rpy="0 0 0"/>
   </joint>
-  <!-- Base link with INCREASED MASS to prevent falling -->
+  <!-- Base link with INCREASED MASS and IMPROVED COLLISION GEOMETRY -->
   <link name="base">
     <inertial>
@@ -104,9 +104,28 @@
       </material>
     </visual>
+    <!-- IMPROVED: Base collision geometry that extends to the bottom -->
     <collision name="base_motor_holder_collision">
-      <origin xyz="0.0206915 0.0221255 0.0300817" rpy="1.5708 0 0"/>
-      <geometry>
-        <box size="0.05 0.05 0.05"/>
-      </geometry>
+      <origin xyz="0.0206915 0.0221255 0.010" rpy="0 0 0"/>
+      <geometry>
+        <box size="0.08 0.08 0.02"/>
+      </geometry>
+      <surface>
+        <friction>
+          <ode>
+            <mu>1.0</mu>
+            <mu2>1.0</mu2>
+          </ode>
+        </friction>
+        <contact>
+          <ode>
+            <soft_cfm>0.0001</soft_cfm>
+            <soft_erp>0.2</soft_erp>
+            <kp>1000000</kp>
+            <kd>100</kd>
+            <max_vel>0.01</max_vel>
+            <min_depth>0.001</min_depth>
+          </ode>
+        </contact>
+      </surface>
     </collision>
     <!-- Base main body visual -->
@@ -120,9 +139,28 @@
       </material>
     </visual>
+    <!-- IMPROVED: Base main collision that provides stable contact -->
     <collision name="base_main_collision">
-      <origin xyz="0.0207909 0.0221255 0.0300817" rpy="1.5708 0 0"/>
-      <geometry>
-        <box size="0.08 0.08 0.08"/>
-      </geometry>
+      <origin xyz="0.0207909 0.0221255 0.030" rpy="0 0 0"/>
+      <geometry>
+        <box size="0.10 0.10 0.06"/>
+      </geometry>
+      <surface>
+        <friction>
+          <ode>
+            <mu>1.0</mu>
+            <mu2>1.0</mu2>
+          </ode>
+        </friction>
+        <contact>
+          <ode>
+            <soft_cfm>0.0001</soft_cfm>
+            <soft_erp>0.2</soft_erp>
+            <kp>1000000</kp>
+            <kd>100</kd>
+            <max_vel>0.01</max_vel>
+            <min_depth>0.001</min_depth>
+          </ode>
+        </contact>
+      </surface>
     </collision>
     <!-- Base motor visual -->
