Commit message: updated project structure

File: urdf/so_arm101.urdf.xacro (robot description, xacro)
@@ -1,9 +1,9 @@
 <?xml version="1.0"?>
-<!-- SO-101 Robot Arm URDF.XACRO for Ignition Gazebo -->
-<robot xmlns:xacro="http://www.ros.org/wiki/xacro" name="so_101_arm">
+<!-- SO-ARM101 Robot Arm URDF.XACRO -->
+<robot xmlns:xacro="http://www.ros.org/wiki/xacro" name="so_arm101">
   <!-- XACRO Parameters -->
-  <xacro:arg name="controller_config_file" default="$(find so_101_arm)/config/controllers_6dof.yaml"/>
+  <xacro:arg name="controller_config_file" default="$(find so_arm101)/config/controllers_6dof.yaml"/>
   <xacro:property name="controller_config" value="$(arg controller_config_file)"/>
-  <!-- ROS2 Control configuration for IGNITION GAZEBO -->
+  <!-- ROS2 Control configuration -->
   <ros2_control name="GazeboSimSystem" type="system">
       <hardware>
@@ -65,5 +65,5 @@
       </joint>
   </ros2_control>
-  <!-- Ignition Gazebo Plugin (NOT Gazebo Classic) -->
+  <!-- Ignition Gazebo Plugin -->
   <gazebo>
     <plugin filename="libgz_ros2_control-system.so" name="gz_ros2_control::GazeboSimROS2ControlPlugin">
@@ -86,9 +86,9 @@
     <origin xyz="0 0 0" rpy="0 0 0"/>
   </joint>
-  <!-- Base link with INCREASED MASS and IMPROVED COLLISION GEOMETRY -->
+  <!-- Base -->
   <link name="base">
     <inertial>
       <origin xyz="0.020739 0.00204287 0.065966" rpy="0 0 0"/>
-      <mass value="50.0"/>  <!-- INCREASED from 0.147 to prevent falling -->
+      <mass value="50.0"/>  <!-- Unrealistic, but essential to keep the arm from tipping over -->
       <inertia ixx="0.136117" ixy="4.59787e-06" ixz="9.75275e-07"
                iyy="0.114686" iyz="-4.97151e-05" izz="0.130364"/>
@@ -98,11 +98,10 @@
       <origin xyz="0.0206915 0.0221255 0.0300817" rpy="1.5708 0 0"/>
       <geometry>
-        <mesh filename="package://so_101_arm/models/so_101_arm/meshes/base_motor_holder_so101_v1.stl"/>
-      </geometry>
-      <material name="plastic">
-        <color rgba="0.1 0.1 0.1 1.0"/>
-      </material>
-    </visual>
-    <!-- IMPROVED: Base collision geometry that extends to the bottom -->
+        <mesh filename="package://chess_robot_sim/models/so_arm101/meshes/base_motor_holder_so101_v1.stl"/>
+      </geometry>
+      <material name="plastic">
+        <color rgba="0.1 0.1 0.1 1.0"/>
+      </material>
+    </visual>
     <collision name="base_motor_holder_collision">
       <origin xyz="0.0206915 0.0221255 0.010" rpy="0 0 0"/>
@@ -133,5 +132,5 @@
       <origin xyz="0.0207909 0.0221255 0.0300817" rpy="1.5708 0 0"/>
       <geometry>
-        <mesh filename="package://so_101_arm/models/so_101_arm/meshes/base_so101_v2.stl"/>
+        <mesh filename="package://chess_robot_sim/models/so_arm101/meshes/base_so101_v2.stl"/>
       </geometry>
       <material name="plastic">
@@ -139,5 +138,4 @@
       </material>
     </visual>
-    <!-- IMPROVED: Base main collision that provides stable contact -->
     <collision name="base_main_collision">
       <origin xyz="0.0207909 0.0221255 0.030" rpy="0 0 0"/>
@@ -168,5 +166,5 @@
       <origin xyz="0.0207909 -0.0105745 0.0761817" rpy="0 0 -1.5708"/>
       <geometry>
-        <mesh filename="package://so_101_arm/models/so_101_arm/meshes/sts3215_03a_v1.stl"/>
+        <mesh filename="package://chess_robot_sim/models/so_arm101/meshes/sts3215_03a_v1.stl"/>
       </geometry>
       <material name="motor">
@@ -184,5 +182,5 @@
       <origin xyz="0.0205915 0.0467435 0.0798817" rpy="1.5708 0 0"/>
       <geometry>
-        <mesh filename="package://so_101_arm/models/so_101_arm/meshes/waveshare_mounting_plate_so101_v2.stl"/>
+        <mesh filename="package://chess_robot_sim/models/so_arm101/meshes/waveshare_mounting_plate_so101_v2.stl"/>
       </geometry>
       <material name="plastic">
@@ -213,5 +211,5 @@
       <origin xyz="-0.0303992 0.000422241 -0.0417" rpy="1.5708 1.5708 0"/>
       <geometry>
-        <mesh filename="package://so_101_arm/models/so_101_arm/meshes/sts3215_03a_v1.stl"/>
+        <mesh filename="package://chess_robot_sim/models/so_arm101/meshes/sts3215_03a_v1.stl"/>
       </geometry>
       <material name="motor">
@@ -229,5 +227,5 @@
       <origin xyz="-0.0675992 -0.000177759 0.0158499" rpy="1.5708 -1.5708 0"/>
       <geometry>
-        <mesh filename="package://so_101_arm/models/so_101_arm/meshes/motor_holder_so101_base_v1.stl"/>
+        <mesh filename="package://chess_robot_sim/models/so_arm101/meshes/motor_holder_so101_base_v1.stl"/>
       </geometry>
       <material name="plastic">
@@ -245,5 +243,5 @@
       <origin xyz="0.0122008 2.22413e-05 0.0464" rpy="-1.5708 0 0"/>
       <geometry>
-        <mesh filename="package://so_101_arm/models/so_101_arm/meshes/rotation_pitch_so101_v1.stl"/>
+        <mesh filename="package://chess_robot_sim/models/so_arm101/meshes/rotation_pitch_so101_v1.stl"/>
       </geometry>
       <material name="plastic">
@@ -283,5 +281,5 @@
       <origin xyz="-0.11257 -0.0155 0.0187" rpy="-3.14159 0 -1.5708"/>
       <geometry>
-        <mesh filename="package://so_101_arm/models/so_101_arm/meshes/sts3215_03a_v1.stl"/>
+        <mesh filename="package://chess_robot_sim/models/so_arm101/meshes/sts3215_03a_v1.stl"/>
       </geometry>
       <material name="motor">
@@ -299,5 +297,5 @@
       <origin xyz="-0.065085 0.012 0.0182" rpy="3.14159 0 0"/>
       <geometry>
-        <mesh filename="package://so_101_arm/models/so_101_arm/meshes/upper_arm_so101_v1.stl"/>
+        <mesh filename="package://chess_robot_sim/models/so_arm101/meshes/upper_arm_so101_v1.stl"/>
       </geometry>
       <material name="plastic">
@@ -337,5 +335,5 @@
       <origin xyz="-0.0648499 -0.032 0.0182" rpy="-3.14159 0 0"/>
       <geometry>
-        <mesh filename="package://so_101_arm/models/so_101_arm/meshes/under_arm_so101_v1.stl"/>
+        <mesh filename="package://chess_robot_sim/models/so_arm101/meshes/under_arm_so101_v1.stl"/>
       </geometry>
       <material name="plastic">
@@ -353,5 +351,5 @@
       <origin xyz="-0.0648499 -0.032 0.018" rpy="-3.14159 0 0"/>
       <geometry>
-        <mesh filename="package://so_101_arm/models/so_101_arm/meshes/motor_holder_so101_wrist_v1.stl"/>
+        <mesh filename="package://chess_robot_sim/models/so_arm101/meshes/motor_holder_so101_wrist_v1.stl"/>
       </geometry>
       <material name="plastic">
@@ -363,5 +361,5 @@
       <origin xyz="-0.1224 0.0052 0.0187" rpy="-3.14159 0 -3.14159"/>
       <geometry>
-        <mesh filename="package://so_101_arm/models/so_101_arm/meshes/sts3215_03a_v1.stl"/>
+        <mesh filename="package://chess_robot_sim/models/so_arm101/meshes/sts3215_03a_v1.stl"/>
       </geometry>
       <material name="motor">
@@ -401,5 +399,5 @@
       <origin xyz="0 -0.0424 0.0306" rpy="1.5708 1.5708 0"/>
       <geometry>
-        <mesh filename="package://so_101_arm/models/so_101_arm/meshes/sts3215_03a_no_horn_v1.stl"/>
+        <mesh filename="package://chess_robot_sim/models/so_arm101/meshes/sts3215_03a_no_horn_v1.stl"/>
       </geometry>
       <material name="motor">
@@ -417,5 +415,5 @@
       <origin xyz="0 -0.028 0.0181" rpy="-1.5708 -1.5708 0"/>
       <geometry>
-        <mesh filename="package://so_101_arm/models/so_101_arm/meshes/wrist_roll_pitch_so101_v2.stl"/>
+        <mesh filename="package://chess_robot_sim/models/so_arm101/meshes/wrist_roll_pitch_so101_v2.stl"/>
       </geometry>
       <material name="plastic">
@@ -455,5 +453,5 @@
       <origin xyz="0.0077 0.0001 -0.0234" rpy="-1.5708 0 0"/>
       <geometry>
-        <mesh filename="package://so_101_arm/models/so_101_arm/meshes/sts3215_03a_v1.stl"/>
+        <mesh filename="package://chess_robot_sim/models/so_arm101/meshes/sts3215_03a_v1.stl"/>
       </geometry>
       <material name="motor">
@@ -471,5 +469,5 @@
       <origin xyz="0 -0.000218214 0.000949706" rpy="-3.14159 0 0"/>
       <geometry>
-        <mesh filename="package://so_101_arm/models/so_101_arm/meshes/wrist_roll_follower_so101_v1.stl"/>
+        <mesh filename="package://chess_robot_sim/models/so_arm101/meshes/wrist_roll_follower_so101_v1.stl"/>
       </geometry>
       <material name="plastic">
@@ -509,5 +507,5 @@
       <origin xyz="0 0 0.0189" rpy="0 0 0"/>
       <geometry>
-        <mesh filename="package://so_101_arm/models/so_101_arm/meshes/moving_jaw_so101_v1.stl"/>
+        <mesh filename="package://chess_robot_sim/models/so_arm101/meshes/moving_jaw_so101_v1.stl"/>
       </geometry>
       <material name="plastic">

Commit message: fixed environment

File: urdf/so_arm101.urdf.xacro (robot description, xacro)
@@ -90,8 +90,33 @@
     <inertial>
       <origin xyz="0.020739 0.00204287 0.065966" rpy="0 0 0"/>
-      <mass value="50.0"/>  <!-- Unrealistic, but essential to keep the arm from tipping over -->
+      <mass value="100.0"/>  <!-- Unrealistic, but essential to keep the arm from tipping over -->
       <inertia ixx="0.136117" ixy="4.59787e-06" ixz="9.75275e-07"
                iyy="0.114686" iyz="-4.97151e-05" izz="0.130364"/>
     </inertial>
+    <!-- Add a more stable base collision -->
+    <collision name="base_stable_collision">
+      <origin xyz="0.0207909 0.0221255 0.010" rpy="0 0 0"/>
+      <geometry>
+        <box size="0.10 0.10 0.02"/>  <!-- Wider, flatter base for better contact -->
+      </geometry>
+      <surface>
+        <friction>
+          <ode>
+            <mu>10.0</mu>   <!-- High friction to prevent sliding -->
+            <mu2>10.0</mu2>
+          </ode>
+        </friction>
+        <contact>
+          <ode>
+            <soft_cfm>0.0001</soft_cfm>
+            <soft_erp>0.2</soft_erp>
+            <kp>1000000</kp>
+            <kd>100</kd>
+            <max_vel>0.01</max_vel>
+            <min_depth>0.001</min_depth>
+          </ode>
+        </contact>
+      </surface>
+    </collision>
     <!-- Base motor holder visual -->
     <visual name="base_motor_holder_visual">
