Commit message: updated spawn position

File: urdf/so_arm_101.urdf.xacro (robot description, xacro)
@@ -194,5 +194,5 @@
     <child link="lower_arm"/>
     <axis xyz="0 0 1"/>
-    <limit lower="-1.74533" upper="1.5708" effort="${joint_effort}" velocity="${joint_velocity}"/>
+    <limit lower="-1.74533" upper="1.74533" effort="${joint_effort}" velocity="${joint_velocity}"/>
     <dynamics damping="0.6" friction="0.052"/>
   </joint>

Commit message: removed floating point ops

File: urdf/so_arm_101.urdf.xacro (robot description, xacro)
@@ -17,10 +17,10 @@
       <origin xyz="0.020739 0.00204287 0.065966" rpy="0 0 0"/>
       <mass value="0.147"/>
-      <inertia ixx="0.000136117" ixy="4.59787e-07" ixz="9.75275e-08"
-               iyy="0.000114686" iyz="-4.97151e-06" izz="0.000130364"/>
+      <inertia ixx="0.0" ixy="0.0" ixz="0.0"
+               iyy="0.0" iyz="0.0" izz="0.0"/>
     </inertial>
     <!-- Base motor holder -->
     <visual>
-      <origin xyz="0.0206915 0.0221255 0.0300817" rpy="1.5708 -1.23909e-16 2.33147e-15"/>
+      <origin xyz="0.0 0.0221255 0.0300817" rpy="1.5708 0.0 0.0"/>
       <geometry>
         <mesh filename="package://so_arm_101_gazebo/meshes/base_motor_holder_so101_v1.stl" scale="${mesh_scale}"/>
@@ -30,5 +30,5 @@
     <!-- Base -->
     <visual>
-      <origin xyz="0.0207909 0.0221255 0.0300817" rpy="1.5708 0 0"/>
+      <origin xyz="0.0 0.0221255 0.0300817" rpy="1.5708 0 0"/>
       <geometry>
         <mesh filename="package://so_arm_101_gazebo/meshes/base_so101_v2.stl" scale="${mesh_scale}"/>
@@ -38,5 +38,5 @@
     <!-- STS3215 Motor -->
     <visual>
-      <origin xyz="0.0207909 -0.0105745 0.0761817" rpy="-2.20282e-15 2.77556e-17 -1.5708"/>
+      <origin xyz="0.0207909 -0.0105745 0.0761817" rpy="0.0 0.0 -1.5708"/>
       <geometry>
         <mesh filename="package://so_arm_101_gazebo/meshes/sts3215_03a_v1.stl" scale="${mesh_scale}"/>
@@ -46,5 +46,5 @@
     <!-- Waveshare mounting plate -->
     <visual>
-      <origin xyz="0.0205915 0.0467435 0.0798817" rpy="1.5708 -1.21716e-14 2.33147e-15"/>
+      <origin xyz="0.0 0.0467435 0.0798817" rpy="1.5708 0.0 0.0"/>
       <geometry>
         <mesh filename="package://so_arm_101_gazebo/meshes/waveshare_mounting_plate_so101_v2.stl" scale="${mesh_scale}"/>
@@ -67,12 +67,12 @@
   <link name="shoulder">
     <inertial>
-      <origin xyz="-0.0307604 -1.66727e-05 -0.0252713" rpy="0 0 0"/>
+      <origin xyz="-0.0307604 0.0 -0.0252713" rpy="0 0 0"/>
       <mass value="0.100006"/>
-      <inertia ixx="8.3759e-05" ixy="7.55525e-08" ixz="-1.16342e-06"
-               iyy="8.10403e-05" iyz="1.54663e-07" izz="2.39783e-05"/>
-    </inertial>
-    <!-- STS3215 Motor -->
-    <visual>
-      <origin xyz="-0.0303992 0.000422241 -0.0417" rpy="1.5708 1.5708 0"/>
+      <inertia ixx="0.0" ixy="0.0" ixz="0.0"
+               iyy="0.0" iyz="0.0" izz="0.0"/>
+    </inertial>
+    <!-- STS3215 Motor -->
+    <visual>
+      <origin xyz="-0.0303992 0.0 -0.0417" rpy="1.5708 1.5708 0"/>
       <geometry>
         <mesh filename="package://so_arm_101_gazebo/meshes/sts3215_03a_v1.stl" scale="${mesh_scale}"/>
@@ -82,5 +82,5 @@
     <!-- Motor holder base -->
     <visual>
-      <origin xyz="-0.0675992 -0.000177759 0.0158499" rpy="1.5708 -1.5708 0"/>
+      <origin xyz="-0.0675992 0.0 0.0158499" rpy="1.5708 -1.5708 0"/>
       <geometry>
         <mesh filename="package://so_arm_101_gazebo/meshes/motor_holder_so101_base_v1.stl" scale="${mesh_scale}"/>
@@ -90,5 +90,5 @@
     <!-- Rotation pitch -->
     <visual>
-      <origin xyz="0.0122008 2.22413e-05 0.0464" rpy="-1.5708 0 0"/>
+      <origin xyz="0.0122008 0.0 0.0464" rpy="-1.5708 0 0"/>
       <geometry>
         <mesh filename="package://so_arm_101_gazebo/meshes/rotation_pitch_so101_v1.stl" scale="${mesh_scale}"/>
@@ -97,5 +97,5 @@
     </visual>
     <collision>
-      <origin xyz="0.0122008 2.22413e-05 0.0464" rpy="-1.5708 0 0"/>
+      <origin xyz="0.0122008 0.0 0.0464" rpy="-1.5708 0 0"/>
       <geometry>
         <mesh filename="package://so_arm_101_gazebo/meshes/rotation_pitch_so101_v1.stl" scale="${mesh_scale}"/>
@@ -104,5 +104,5 @@
   </link>
   <joint name="shoulder_rotation" type="revolute">
-    <origin xyz="0.0207909 -0.0230745 0.0948817" rpy="-3.14159 6.03684e-16 1.5708"/>
+    <origin xyz="0.0 -0.0230745 0.0948817" rpy="-3.14159 0.0 1.5708"/>
     <parent link="base"/>
     <child link="shoulder"/>
@@ -116,10 +116,10 @@
       <origin xyz="-0.0898471 -0.00838224 0.0184089" rpy="0 0 0"/>
       <mass value="0.103"/>
-      <inertia ixx="4.08002e-05" ixy="-1.97819e-05" ixz="-4.03016e-08"
-               iyy="0.000147318" iyz="8.97326e-09" izz="0.000142487"/>
-    </inertial>
-    <!-- STS3215 Motor -->
-    <visual>
-      <origin xyz="-0.11257 -0.0155 0.0187" rpy="-3.14159 -6.8695e-16 -1.5708"/>
+      <inertia ixx="0.0" ixy="0.0" ixz="0.0"
+               iyy="0.0" iyz="0.0" izz="0.0"/>
+    </inertial>
+    <!-- STS3215 Motor -->
+    <visual>
+      <origin xyz="-0.11257 -0.0155 0.0187" rpy="-3.14159 0.0 -1.5708"/>
       <geometry>
         <mesh filename="package://so_arm_101_gazebo/meshes/sts3215_03a_v1.stl" scale="${mesh_scale}"/>
@@ -129,5 +129,5 @@
     <!-- Upper arm -->
     <visual>
-      <origin xyz="-0.065085 0.012 0.0182" rpy="3.14159 -9.35612e-32 0"/>
+      <origin xyz="-0.065085 0.012 0.0182" rpy="3.14159 0.0 0"/>
       <geometry>
         <mesh filename="package://so_arm_101_gazebo/meshes/upper_arm_so101_v1.stl" scale="${mesh_scale}"/>
@@ -136,5 +136,5 @@
     </visual>
     <collision>
-      <origin xyz="-0.065085 0.012 0.0182" rpy="3.14159 -9.35612e-32 0"/>
+      <origin xyz="-0.065085 0.012 0.0182" rpy="3.14159 0.0 0"/>
       <geometry>
         <mesh filename="package://so_arm_101_gazebo/meshes/upper_arm_so101_v1.stl" scale="${mesh_scale}"/>
@@ -155,10 +155,10 @@
       <origin xyz="-0.0980701 0.00324376 0.0182831" rpy="0 0 0"/>
       <mass value="0.104"/>
-      <inertia ixx="2.87438e-05" ixy="7.41152e-06" ixz="1.26409e-06"
-               iyy="0.000159844" iyz="-4.90188e-08" izz="0.00014529"/>
+      <inertia ixx="0.0" ixy="0.0" ixz="0.0"
+               iyy="0.0" iyz="0.0" izz="0.0"/>
     </inertial>
     <!-- Under arm -->
     <visual>
-      <origin xyz="-0.0648499 -0.032 0.0182" rpy="-3.14159 0 3.9443e-31"/>
+      <origin xyz="-0.0648499 -0.032 0.0182" rpy="-3.14159 0 0.0"/>
       <geometry>
         <mesh filename="package://so_arm_101_gazebo/meshes/under_arm_so101_v1.stl" scale="${mesh_scale}"/>
@@ -168,5 +168,5 @@
     <!-- Motor holder wrist -->
     <visual>
-      <origin xyz="-0.0648499 -0.032 0.018" rpy="-3.14159 4.73317e-30 7.88861e-31"/>
+      <origin xyz="-0.0648499 -0.032 0.018" rpy="-3.14159 0.0 0.0"/>
       <geometry>
         <mesh filename="package://so_arm_101_gazebo/meshes/motor_holder_so101_wrist_v1.stl" scale="${mesh_scale}"/>
@@ -176,12 +176,12 @@
     <!-- STS3215 Motor -->
     <visual>
-      <origin xyz="-0.1224 0.0052 0.0187" rpy="-3.14159 -3.58047e-15 -3.14159"/>
-      <geometry>
-        <mesh filename="package://so_arm_101_gazebo/meshes/sts3215_03a_v1.stl" scale="${mesh_scale}"/>
-      </geometry>
-      <material name="so101_metal"/>
-    </visual>
-    <collision>
-      <origin xyz="-0.0648499 -0.032 0.0182" rpy="-3.14159 0 3.9443e-31"/>
+      <origin xyz="-0.1224 0.0052 0.0187" rpy="-3.14159 0.0 -3.14159"/>
+      <geometry>
+        <mesh filename="package://so_arm_101_gazebo/meshes/sts3215_03a_v1.stl" scale="${mesh_scale}"/>
+      </geometry>
+      <material name="so101_metal"/>
+    </visual>
+    <collision>
+      <origin xyz="-0.0648499 -0.032 0.0182" rpy="-3.14159 0 0.0"/>
       <geometry>
         <mesh filename="package://so_arm_101_gazebo/meshes/under_arm_so101_v1.stl" scale="${mesh_scale}"/>
@@ -190,5 +190,5 @@
   </link>
   <joint name="elbow" type="revolute">
-    <origin xyz="-0.11257 -0.028 2.46331e-16" rpy="-1.22818e-15 5.75928e-16 1.5708"/>
+    <origin xyz="-0.11257 -0.028 0.0" rpy="0.0 0.0 1.5708"/>
     <parent link="upper_arm"/>
     <child link="lower_arm"/>
@@ -200,12 +200,12 @@
   <link name="wrist">
     <inertial>
-      <origin xyz="-0.000103312 -0.0386143 0.0281156" rpy="0 0 0"/>
+      <origin xyz="0.0 -0.0386143 0.0281156" rpy="0 0 0"/>
       <mass value="0.079"/>
-      <inertia ixx="3.68263e-05" ixy="1.7893e-08" ixz="-5.28128e-08"
-               iyy="2.5391e-05" iyz="3.6412e-06" izz="2.1e-05"/>
+      <inertia ixx="0.0" ixy="0.0" ixz="0.0"
+               iyy="0.0" iyz="0.0" izz="0.0"/>
     </inertial>
     <!-- STS3215 Motor no horn -->
     <visual>
-      <origin xyz="5.55112e-17 -0.0424 0.0306" rpy="1.5708 1.5708 0"/>
+      <origin xyz="0.0 -0.0424 0.0306" rpy="1.5708 1.5708 0"/>
       <geometry>
         <mesh filename="package://so_arm_101_gazebo/meshes/sts3215_03a_no_horn_v1.stl" scale="${mesh_scale}"/>
@@ -229,5 +229,5 @@
   </link>
   <joint name="wrist_pitch" type="revolute">
-    <origin xyz="-0.1349 0.0052 1.65232e-16" rpy="3.2474e-15 2.86219e-15 -1.5708"/>
+    <origin xyz="-0.1349 0.0052 0.0" rpy="0.0 0.0 -1.5708"/>
     <parent link="lower_arm"/>
     <child link="wrist"/>
@@ -239,12 +239,12 @@
   <link name="gripper">
     <inertial>
-      <origin xyz="0.000213627 0.000245138 -0.025187" rpy="0 0 0"/>
+      <origin xyz="0.0 0.0 -0.025187" rpy="0 0 0"/>
       <mass value="0.087"/>
-      <inertia ixx="2.75087e-05" ixy="-3.35241e-07" ixz="-5.7352e-06"
-               iyy="4.33657e-05" iyz="-5.17847e-08" izz="3.45059e-05"/>
-    </inertial>
-    <!-- STS3215 Motor -->
-    <visual>
-      <origin xyz="0.0077 0.0001 -0.0234" rpy="-1.5708 -5.55112e-17 -1.38213e-14"/>
+      <inertia ixx="0.0" ixy="0.0" ixz="0.0"
+               iyy="0.0" iyz="0.0" izz="0.0"/>
+    </inertial>
+    <!-- STS3215 Motor -->
+    <visual>
+      <origin xyz="0.0077 0.0 -0.0234" rpy="-1.5708 0.0 0.0"/>
       <geometry>
         <mesh filename="package://so_arm_101_gazebo/meshes/sts3215_03a_v1.stl" scale="${mesh_scale}"/>
@@ -254,5 +254,5 @@
     <!-- Wrist roll follower -->
     <visual>
-      <origin xyz="5.55112e-17 -0.000218214 0.000949706" rpy="-3.14159 -5.55112e-17 -9.17912e-24"/>
+      <origin xyz="0.0 0.0 0.0" rpy="-3.14159 0.0 0.0"/>
       <geometry>
         <mesh filename="package://so_arm_101_gazebo/meshes/wrist_roll_follower_so101_v1.stl" scale="${mesh_scale}"/>
@@ -261,5 +261,5 @@
     </visual>
     <collision>
-      <origin xyz="5.55112e-17 -0.000218214 0.000949706" rpy="-3.14159 -5.55112e-17 -9.17912e-24"/>
+      <origin xyz="0.0 0.0 0.0" rpy="-3.14159 0.0 0.0"/>
       <geometry>
         <mesh filename="package://so_arm_101_gazebo/meshes/wrist_roll_follower_so101_v1.stl" scale="${mesh_scale}"/>
@@ -268,5 +268,5 @@
   </link>
   <joint name="wrist_roll" type="revolute">
-    <origin xyz="0 -0.0611 0.0181" rpy="1.5708 -9.38083e-08 3.14159"/>
+    <origin xyz="0 -0.0611 0.0181" rpy="1.5708 0.0 3.14159"/>
     <parent link="wrist"/>
     <child link="gripper"/>
@@ -280,10 +280,10 @@
       <origin xyz="-0.00157495 -0.0300244 0.0192755" rpy="0 0 0"/>
       <mass value="0.012"/>
-      <inertia ixx="6.61427e-06" ixy="-3.19807e-07" ixz="-5.90717e-09"
-               iyy="1.89032e-06" iyz="-1.09945e-07" izz="5.28738e-06"/>
+      <inertia ixx="0.0" ixy="0.0" ixz="0.0"
+               iyy="0.0" iyz="0.0" izz="0.0"/>
     </inertial>
     <!-- Moving jaw -->
     <visual>
-      <origin xyz="-5.55112e-17 -1.94746e-17 0.0189" rpy="9.53145e-17 -4.66093e-24 0"/>
+      <origin xyz="0.0 0.0 0.0189" rpy="0.0 0.0 0"/>
       <geometry>
         <mesh filename="package://so_arm_101_gazebo/meshes/moving_jaw_so101_v1.stl" scale="${mesh_scale}"/>
@@ -292,5 +292,5 @@
     </visual>
     <collision>
-      <origin xyz="-5.55112e-17 -1.94746e-17 0.0189" rpy="9.53145e-17 -4.66093e-24 0"/>
+      <origin xyz="0.0 0.0 0.0189" rpy="0.0 0.0 0"/>
       <geometry>
         <mesh filename="package://so_arm_101_gazebo/meshes/moving_jaw_so101_v1.stl" scale="${mesh_scale}"/>
@@ -299,5 +299,5 @@
   </link>
   <joint name="gripper_joint" type="revolute">
-    <origin xyz="0.0202 0.0188 -0.0234" rpy="1.5708 -5.14108e-17 -1.38655e-14"/>
+    <origin xyz="0.0202 0.0188 -0.0234" rpy="1.5708 0.0 0.0"/>
     <parent link="gripper"/>
     <child link="gripper_jaw"/>
